File: HW2/pcb1.brd (EAGLE design)
At the start: 50 x 50 mm, 22 parts, among them J1 USB-MB-H

Commit message: brd
first try of layout - pre error check
Parts:
- moved C2 25.0 mm to (18.9, 9.67)
- moved U$7 6.40 mm to (18.2, 18.9)
- moved R1 3.61 mm to (42.1, 40.6)
- moved R4 3.00 mm to (6.55, 11.7)
- moved R3 2.00 mm to (13.2, 11.7)
- moved C4 1.00 mm to (34.5, 44.3)
- moved U$4 1.00 mm to (17.0, 3.24)

Commit message: Made a pcb
made some gerber files
Parts:
- moved U$4 7.07 mm to (24.0, 2.24)
- moved U$5 7.00 mm to (15.2, 2.67)
- moved LED2 6.00 mm to (32.4, 3.07)
- moved R4 5.00 mm to (11.6, 11.7)
- moved R2 4.92 mm to (39.2, 7.63)
- moved J2 4.34 mm to (1.27, 16.5)
- moved U$6 4.00 mm to (1.71, 13.6)
- moved C5 1.41 mm to (35.1, 20.3)
- moved C1 1.00 mm to (33.8, 39.7)
- moved C2 1.00 mm to (18.9, 8.67), turned to 270 degrees
- moved C3 1.00 mm to (35.0, 48.7)
- moved R1 1.00 mm to (42.1, 39.6)
- moved R3 1.00 mm to (14.2, 11.7)
- moved U$1 1.00 mm to (27.2, 24.4)
- moved J3 0.82 mm to (48.8, 16.5)
Routing:
- net +3V3: track 0.00 -> 128.1 mm, vias 0 -> 6
- net +5V: track 0.00 -> 100.6 mm, vias 0 -> 5
- net MCLR: track 0.00 -> 63.8 mm, vias 0 -> 2
- net B4/USER: track 0.00 -> 58.1 mm, vias 0 -> 2
- net USBID: track 0.00 -> 56.2 mm, vias 0 -> 2
- net PGC: track 0.00 -> 49.9 mm, vias 0 -> 2
- net PGD: track 0.00 -> 48.9 mm, vias 0 -> 2
- net D+: track 0.00 -> 46.1 mm, vias 0 -> 2
- net A4/LED: track 0.00 -> 45.1 mm, vias 0 -> 3
- net D-: track 0.00 -> 43.0 mm, vias 0 -> 1
- net A1: track 0.00 -> 24.0 mm
- net A0: track 0.00 -> 23.8 mm
- net B3: track 0.00 -> 22.6 mm
- net B2: track 0.00 -> 22.6 mm
- net B9: track 0.00 -> 22.4 mm
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- added copper zone on layer 16, net GND
